Commit message: home-up named xarm pose

File: xarm_moveit_config/srdf/_xarm7_macro.srdf.xacro (robot description, xacro)
@@ -57,4 +57,13 @@
       <joint name="${prefix}joint6" value="-1.5708" />
       <joint name="${prefix}joint7" value="0" />
+    </group_state>
+    <group_state name="home-up" group="${prefix}xarm7">
+      <joint name="${prefix}joint1" value="0" />
+      <joint name="${prefix}joint2" value="-0.975" />
+      <joint name="${prefix}joint3" value="0" />
+      <joint name="${prefix}joint4" value="0.58" />
+      <joint name="${prefix}joint5" value="0" />
+      <joint name="${prefix}joint6" value="1.57" />
+      <joint name="${prefix}joint7" value="0.0" />
     </group_state>
     <!-- gripper -->

Commit message: hold right named goal

File: xarm_moveit_config/srdf/_xarm7_macro.srdf.xacro (robot description, xacro)
@@ -66,4 +66,13 @@
       <joint name="${prefix}joint6" value="1.57" />
       <joint name="${prefix}joint7" value="0.0" />
+    </group_state>
+    <group_state name="hold-right" group="${prefix}xarm7">
+      <joint name="${prefix}joint1" value="-0.5" />
+      <joint name="${prefix}joint2" value="-0.02" />
+      <joint name="${prefix}joint3" value="-0.27" />
+      <joint name="${prefix}joint4" value="0.35" />
+      <joint name="${prefix}joint5" value="0.85" />
+      <joint name="${prefix}joint6" value="1.825" />
+      <joint name="${prefix}joint7" value="0.275" />
     </group_state>
     <!-- gripper -->

Commit message: named goal update

File: xarm_moveit_config/srdf/_xarm7_macro.srdf.xacro (robot description, xacro)
@@ -68,11 +68,11 @@
     </group_state>
     <group_state name="hold-right" group="${prefix}xarm7">
-      <joint name="${prefix}joint1" value="-0.5" />
-      <joint name="${prefix}joint2" value="-0.02" />
-      <joint name="${prefix}joint3" value="-0.27" />
-      <joint name="${prefix}joint4" value="0.35" />
-      <joint name="${prefix}joint5" value="0.85" />
-      <joint name="${prefix}joint6" value="1.825" />
-      <joint name="${prefix}joint7" value="0.275" />
+      <joint name="${prefix}joint1" value="-0.525" />
+      <joint name="${prefix}joint2" value="-0.398" />
+      <joint name="${prefix}joint3" value="-0.28" />
+      <joint name="${prefix}joint4" value="0.355" />
+      <joint name="${prefix}joint5" value="0.89" />
+      <joint name="${prefix}joint6" value="2.01" />
+      <joint name="${prefix}joint7" value="0.64" />
     </group_state>
     <!-- gripper -->

Commit message: hold-up2 named goal

File: xarm_moveit_config/srdf/_xarm7_macro.srdf.xacro (robot description, xacro)
@@ -67,12 +67,12 @@
       <joint name="${prefix}joint7" value="0.0" />
     </group_state>
-    <group_state name="hold-right" group="${prefix}xarm7">
-      <joint name="${prefix}joint1" value="-0.525" />
-      <joint name="${prefix}joint2" value="-0.398" />
-      <joint name="${prefix}joint3" value="-0.28" />
-      <joint name="${prefix}joint4" value="0.355" />
-      <joint name="${prefix}joint5" value="0.89" />
-      <joint name="${prefix}joint6" value="2.01" />
-      <joint name="${prefix}joint7" value="0.64" />
+    <group_state name="hold-up2" group="${prefix}xarm7">
+      <joint name="${prefix}joint1" value="0.0" />
+      <joint name="${prefix}joint2" value="-0.89" />
+      <joint name="${prefix}joint3" value="0.0" />
+      <joint name="${prefix}joint4" value="0.28" />
+      <joint name="${prefix}joint5" value="3.141" />
+      <joint name="${prefix}joint6" value="0.387" />
+      <joint name="${prefix}joint7" value="0.0" />
     </group_state>
     <!-- gripper -->

Commit message: hold-up60 named pose

File: xarm_moveit_config/srdf/_xarm7_macro.srdf.xacro (robot description, xacro)
@@ -69,10 +69,19 @@
     <group_state name="hold-up2" group="${prefix}xarm7">
       <joint name="${prefix}joint1" value="0.0" />
-      <joint name="${prefix}joint2" value="-0.89" />
+      <joint name="${prefix}joint2" value="-0.743" />
       <joint name="${prefix}joint3" value="0.0" />
-      <joint name="${prefix}joint4" value="0.28" />
-      <joint name="${prefix}joint5" value="3.141" />
-      <joint name="${prefix}joint6" value="0.387" />
+      <joint name="${prefix}joint4" value="0.1" />
+      <joint name="${prefix}joint5" value="3.14" />
+      <joint name="${prefix}joint6" value="0.7" />
       <joint name="${prefix}joint7" value="0.0" />
+    </group_state>
+    <group_state name="hold-up60" group="${prefix}xarm7">
+      <joint name="${prefix}joint1" value="-0.0375" />
+      <joint name="${prefix}joint2" value="-0.4377" />
+      <joint name="${prefix}joint3" value="-0.7255" />
+      <joint name="${prefix}joint4" value="0.315" />
+      <joint name="${prefix}joint5" value="1.234" />
+      <joint name="${prefix}joint6" value="1.466" />
+      <joint name="${prefix}joint7" value="0.707" />
     </group_state>
     <!-- gripper -->
